Commit message: test remote

File: description/camera.xacro (robot description, xacro)
@@ -9,5 +9,5 @@
         <visual>
             <geometry>
-                <box size="0.010 0.03 0.03"/>
+                <box size="0.015 0.03 0.03"/>
             </geometry>
             <material name="red"/>
