Commit message: fix size

File: description/gazebo_control.xacro (robot description, xacro)
@@ -6,6 +6,6 @@
             <left_joint>left_wheel_joint</left_joint>
             <right_joint>right_wheel_joint</right_joint>
-            <wheel_separation>0.297</wheel_separation>
-            <wheel_diameter>0.066</wheel_diameter>
+            <wheel_separation>0.18</wheel_separation>
+            <wheel_diameter>0.035</wheel_diameter>
             <!-- Limits -->
             <max_wheel_torque>200</max_wheel_torque>

File: description/robot_core.xacro (robot description, xacro)
@@ -65,5 +65,5 @@
         <visual>
             <geometry>
-                <cylinder radius="0.034" length="0.0254"/>
+                <cylinder radius="0.035" length="0.0254"/>
             </geometry>
             <material name="blue"/>
@@ -71,8 +71,8 @@
         <collision>
             <geometry>
-                <sphere radius="0.034"/>
+                <sphere radius="0.035"/>
             </geometry>
         </collision>
-        <xacro:inertial_cylinder mass="0.1" length="0.0254" radius="0.034">
+        <xacro:inertial_cylinder mass="0.1" length="0.0254" radius="0.035">
             <origin xyz="0 0 0" rpy="0 0 0"/>
         </xacro:inertial_cylinder>
@@ -91,5 +91,5 @@
         <visual>
             <geometry>
-                <cylinder radius="0.034" length="0.0254"/>
+                <cylinder radius="0.035" length="0.0254"/>
             </geometry>
             <material name="blue"/>
@@ -97,8 +97,8 @@
         <collision>
             <geometry>
-                <sphere radius="0.034"/>
+                <sphere radius="0.035"/>
             </geometry>
         </collision>
-        <xacro:inertial_cylinder mass="0.1" length="0.0254" radius="0.034">
+        <xacro:inertial_cylinder mass="0.1" length="0.0254" radius="0.035">
             <origin xyz="0 0 0" rpy="0 0 0"/>
         </xacro:inertial_cylinder>
